Commit message: the whole arm

File: urdf/mrm.xacro (robot description, xacro)
@@ -13,6 +13,6 @@
 	<joint name="base_link__link_01" type="revolute">
            <axis xyz="0 0 1" />
-           <limit effort="1000.0" lower="-3.14" upper="0.5" velocity="0.5" /> <!--  The lower and upper values define by how much we can rotate.   -->
-           <origin rpy="0 0 0" xyz="0 0 0.5" />
+           <limit effort="1000.0" lower="-3.14" upper="3.14" velocity="0.5" /> <!--  The lower and upper values define by how much we can rotate.   -->
+           <origin rpy="0 0 0" xyz="0 0 0.5" /> <!-- half of the height of the box- base_link -->
            <parent link="base_link" />
            <child link="link_01" />
@@ -26,3 +26,67 @@
 		</visual>
 	</link>
+<!-- between the links there has to be a joint -->
+	<joint name="link_01__link_02" type="revolute">
+           <axis xyz="0 1 0" />
+           <limit effort="1000.0" lower="0" upper="0.5" velocity="0.5" /> <!--  The lower and upper values define by how much we can rotate.   -->
+           <origin rpy="0 0 0" xyz="0 0 0.4" /> <!-- half of the height of the box- base_link -->
+           <parent link="link_01" />
+           <child link="link_02" />
+    </joint>
+	<link name  = "link_02">
+		<visual>
+			<origin rpy = "0 0 0" xyz = "0 0 0.4"/>
+			<geometry>
+				<cylinder radius  = "0.15" length = "0.8"/>
+			</geometry>
+		</visual>
+	</link>
+<!-- between the links there has to be a joint -->
+	<joint name="link_02__link_03" type="revolute">
+           <axis xyz="0 1 0" />
+           <limit effort="1000.0" lower="0" upper="0.75" velocity="0.5" /> <!--  The lower and upper values define by how much we can rotate.   -->
+           <origin rpy="0 0 0" xyz="0 0 0.8" /> <!-- half of the height of the box- base_link -->
+           <parent link="link_02" />
+           <child link="link_03" />
+    </joint>
+	<link name  = "link_03">
+		<visual>
+			<origin rpy = "0 0 0" xyz = "0 0 0.4"/>
+			<geometry>
+				<cylinder radius  = "0.15" length = "0.8"/>
+			</geometry>
+		</visual>
+	</link>
+<!-- between the links there has to be a joint -->
+	<joint name="link_03__link_04" type="revolute">
+           <axis xyz="0 1 0" />
+           <limit effort="1000.0" lower="0" upper="0.75" velocity="0.5" /> <!--  The lower and upper values define by how much we can rotate.   -->
+           <origin rpy="0 0 0" xyz="0 0 0.8" /> <!-- half of the height of the box- base_link -->
+           <parent link="link_03" />
+           <child link="link_04" />
+    </joint>
+	<link name  = "link_04">
+		<visual>
+			<origin rpy = "0 0 0" xyz = "0 0 0.4"/>
+			<geometry>
+				<cylinder radius  = "0.15" length = "0.8"/>
+			</geometry>
+		</visual>
+	</link>
+<!-- between the links there has to be a joint -->
+	<joint name="link_04__link_05" type="revolute">
+           <axis xyz="0 0 1" />
+           <limit effort="1000.0" lower="-3.14" upper="3.14" velocity="0.5" /> <!--  The lower and upper values define by how much we can rotate.   -->
+           <origin rpy="0 0 0" xyz="0 0 0.8" /> <!-- half of the height of the box- base_link -->
+           <parent link="link_04" />
+           <child link="link_05" />
+    </joint>
+	<link name  = "link_05">
+		<visual>
+			<origin rpy = "0 0 0" xyz = "0 0 0.125"/>
+			<geometry>
+				<cylinder radius  = "0.15" length = "0.25"/>
+			</geometry>
+		</visual>
+	</link>
 </robot>

Commit message: finished adding controllers for the arm

File: urdf/mrm.xacro (robot description, xacro)
@@ -1,92 +1,79 @@
 <?xml version = "1.0" ?>
 <robot name ="mrm" xmlns:xacro="http://www.ros.org/wiki/xacro">
+	<xacro:include filename="$(find mrm_decsription)/urdf/robot_parameters.xacro" />
+	<xacro:include filename="$(find mrm_decsription)/urdf/links_joints.xacro" />
 <!-- this is fixed -->
-	<link name  = "base_link">
-		<visual>
-			<origin rpy = "0 0 0" xyz = "0 0 0"/>
-			<geometry>
-				<box size = "1 1 1" />
-			</geometry>
-		</visual>
-	</link>
+	<m_link_box name="${link_00_name}"
+              origin_rpy="0 0 0" origin_xyz="0 0 0"
+              mass="1024"
+              ixx="170.667" ixy="0" ixz="0"
+              iyy="170.667" iyz="0"
+              izz="170.667"
+              size="1 1 1" />
 <!-- between the links there has to be a joint -->
-	<joint name="base_link__link_01" type="revolute">
-           <axis xyz="0 0 1" />
-           <limit effort="1000.0" lower="-3.14" upper="3.14" velocity="0.5" /> <!--  The lower and upper values define by how much we can rotate.   -->
-           <origin rpy="0 0 0" xyz="0 0 0.5" /> <!-- half of the height of the box- base_link -->
-           <parent link="base_link" />
-           <child link="link_01" />
-    </joint>
-	<link name  = "link_01">
-		<visual>
-			<origin rpy = "0 0 0" xyz = "0 0 0.2"/>
-			<geometry>
-				<cylinder radius  = "0.35" length = "0.4"/>
-			</geometry>
-		</visual>
-	</link>
-<!-- between the links there has to be a joint -->
-	<joint name="link_01__link_02" type="revolute">
-           <axis xyz="0 1 0" />
-           <limit effort="1000.0" lower="0" upper="0.5" velocity="0.5" /> <!--  The lower and upper values define by how much we can rotate.   -->
-           <origin rpy="0 0 0" xyz="0 0 0.4" /> <!-- half of the height of the box- base_link -->
-           <parent link="link_01" />
-           <child link="link_02" />
-    </joint>
-	<link name  = "link_02">
-		<visual>
-			<origin rpy = "0 0 0" xyz = "0 0 0.4"/>
-			<geometry>
-				<cylinder radius  = "0.15" length = "0.8"/>
-			</geometry>
-		</visual>
-	</link>
-<!-- between the links there has to be a joint -->
-	<joint name="link_02__link_03" type="revolute">
-           <axis xyz="0 1 0" />
-           <limit effort="1000.0" lower="0" upper="0.75" velocity="0.5" /> <!--  The lower and upper values define by how much we can rotate.   -->
-           <origin rpy="0 0 0" xyz="0 0 0.8" /> <!-- half of the height of the box- base_link -->
-           <parent link="link_02" />
-           <child link="link_03" />
-    </joint>
-	<link name  = "link_03">
-		<visual>
-			<origin rpy = "0 0 0" xyz = "0 0 0.4"/>
-			<geometry>
-				<cylinder radius  = "0.15" length = "0.8"/>
-			</geometry>
-		</visual>
-	</link>
-<!-- between the links there has to be a joint -->
-	<joint name="link_03__link_04" type="revolute">
-           <axis xyz="0 1 0" />
-           <limit effort="1000.0" lower="0" upper="0.75" velocity="0.5" /> <!--  The lower and upper values define by how much we can rotate.   -->
-           <origin rpy="0 0 0" xyz="0 0 0.8" /> <!-- half of the height of the box- base_link -->
-           <parent link="link_03" />
-           <child link="link_04" />
-    </joint>
-	<link name  = "link_04">
-		<visual>
-			<origin rpy = "0 0 0" xyz = "0 0 0.4"/>
-			<geometry>
-				<cylinder radius  = "0.15" length = "0.8"/>
-			</geometry>
-		</visual>
-	</link>
-<!-- between the links there has to be a joint -->
-	<joint name="link_04__link_05" type="revolute">
-           <axis xyz="0 0 1" />
-           <limit effort="1000.0" lower="-3.14" upper="3.14" velocity="0.5" /> <!--  The lower and upper values define by how much we can rotate.   -->
-           <origin rpy="0 0 0" xyz="0 0 0.8" /> <!-- half of the height of the box- base_link -->
-           <parent link="link_04" />
-           <child link="link_05" />
-    </joint>
-	<link name  = "link_05">
-		<visual>
-			<origin rpy = "0 0 0" xyz = "0 0 0.125"/>
-			<geometry>
-				<cylinder radius  = "0.15" length = "0.25"/>
-			</geometry>
-		</visual>
-	</link>
+	<m_joint name="${link_00_name}__${link_01_name}" type="revolute"
+           axis_xyz="0 0 1"
+           origin_rpy="0 0 0" origin_xyz="0 0 0.5"
+           parent="base_link" child="link_01"
+           limit_e="1000" limit_l="-3.14" limit_u="3.14" limit_v="0.5" />
+	 <m_link_mesh name="${link_01_name}"
+              origin_rpy="0 0 0" origin_xyz="0 0 -0.1"
+              mass="157.633"
+              ixx="13.235" ixy="0" ixz="0"
+              iyy="13.235" iyz="0"
+              izz="9.655"
+              meshfile="package://mrm_decsription/meshes/Link1-v2.stl"
+              meshscale="0.001 0.001 0.001" />
+	<m_joint name="${link_01_name}__${link_02_name}" type="revolute"
+           axis_xyz="0 1 0"
+           origin_rpy="0 0 0" origin_xyz="0 0 0.4"
+           parent="link_01" child="link_02"
+           limit_e="1000" limit_l="0" limit_u="0.5" limit_v="0.5" />
+  <m_link_cylinder name="${link_02_name}"
+              origin_rpy="0 0 0" origin_xyz="0 0 0.4"
+              mass="57.906"
+              ixx="12.679" ixy="0" ixz="0"
+              iyy="12.679" iyz="0"
+              izz="0.651"
+              radius="0.15" length="0.8" />
+	 <m_joint name="${link_02_name}__${link_03_name}" type="revolute"
+           axis_xyz="0 1 0"
+           origin_rpy="0 0 0" origin_xyz="0 0 0.8"
+           parent="link_02" child="link_03"
+           limit_e="1000" limit_l="0" limit_u="0.75" limit_v="0.5" />
+  <m_link_cylinder name="${link_03_name}"
+              origin_rpy="0 0 0" origin_xyz="0 0 0.4"
+              mass="57.906"
+              ixx="12.679" ixy="0" ixz="0"
+              iyy="12.679" iyz="0"
+              izz="0.651"
+              radius="0.15" length="0.8" />
+	<m_joint name="${link_03_name}__${link_04_name}" type="revolute"
+           axis_xyz="0 1 0"
+           origin_rpy="0 0 0" origin_xyz="0 0 0.8"
+           parent="link_03" child="link_04"
+           limit_e="1000" limit_l="0" limit_u="0.75" limit_v="0.5" />
+    <m_link_cylinder name="${link_04_name}"
+              origin_rpy="0 0 0" origin_xyz="0 0 0.4"
+              mass="57.906"
+              ixx="12.679" ixy="0" ixz="0"
+              iyy="12.679" iyz="0"
+              izz="0.651"
+              radius="0.15" length="0.8" />
+	<m_joint name="${link_04_name}__${link_05_name}" type="revolute"
+           axis_xyz="0 0 1"
+           origin_rpy="0 0 0" origin_xyz="0 0 0.8"
+           parent="link_04" child="link_05"
+           limit_e="1000" limit_l="-3.14" limit_u="3.14" limit_v="0.5" />
+    <m_link_cylinder name="${link_05_name}"
+              origin_rpy="0 0 0" origin_xyz="0 0 0.125"
+              mass="18.056"
+              ixx="0.479" ixy="0" ixz="0"
+              iyy="0.479" iyz="0"
+              izz="0.204"
+              radius="0.15" length="0.25" />
+    <gazebo>
+    <plugin name="gazebo_ros_control" filename="libgazebo_ros_control.so">
+    </plugin>
+  </gazebo>
 </robot>
