Commit message: new changes to color

File: urdf/links_joints.xacro (robot description, xacro)
@@ -1,4 +1,16 @@
 <?xml version="1.0" ?>
 <robot xmlns:xacro="http://www.ros.org/wiki/xacro">
+<material name="blue">
+    <color rgba="0 0 0.8 1"/>
+  </material>
+  <material name="white">
+    <color rgba="1 1 1 1"/>
+  </material>
+  <material name="black">
+    <color rgba="0 0 0 0"/>
+  </material>
+  <material name="cyan">
+    <color rgba="0 0.9 0.9 1.0"/>
+  </material>
   <xacro:macro name="m_joint" params="name type axis_xyz origin_rpy origin_xyz parent child limit_e limit_l limit_u limit_v">
     <joint name="${name}" type="${type}">
@@ -38,4 +50,5 @@
           <cylinder radius="${radius}" length="${length}" />
         </geometry>
+        <material name="cyan"/>
       </visual>
     </link>
@@ -59,4 +72,5 @@
           <box size="${size}" />
         </geometry>
+        <material name="blue"/>
       </visual>
     </link>

File: urdf/mrm.xacro (robot description, xacro)
@@ -25,5 +25,5 @@
               meshfile="package://mrm_decsription/meshes/Link1-v2.stl"
               meshscale="0.001 0.001 0.001" />
-	<m_joint name="${link_01_name}__${link_02_name}" type="revolute"
+	<m_joint name="${link_00_name}__${link_02_name}" type="revolute"
            axis_xyz="0 1 0"
            origin_rpy="0 0 0" origin_xyz="0 0 0.4"
@@ -73,7 +73,75 @@
               izz="0.204"
               radius="0.15" length="0.25" />
+<!-- camera link and joint -->
+    <joint name="camera_joint" type="fixed">
+    	<axis xyz="0 1 0" />
+    	<origin rpy="0 0 0" xyz="0.7 0 0"/>
+    	<parent link="${link_00_name}"/>
+    	<child link="camera_link"/>
+  	</joint>
+ 	 <!-- Camera -->
+  	<link name="camera_link">
+    	<collision>
+      		<origin xyz="0.5 0 0" rpy="0 0 0"/>
+      		<geometry>
+    			<box size="${camera_link} ${camera_link} ${camera_link}"/>
+      		</geometry>
+    	</collision>
+    	<visual>
+      		<origin xyz="0 0 0" rpy="0 0 0"/>
+      		<geometry>
+    			<box size="${camera_link} ${camera_link} ${camera_link}"/>
+      		</geometry>
+    	</visual>
+    	<inertial>
+      		<mass value="1e-5" />
+      		<origin xyz="0 0 0" rpy="0 0 0"/>
+      		<inertia ixx="1e-6" ixy="0" ixz="0" iyy="1e-6" iyz="0" izz="1e-6" />
+    	</inertial>
+  </link>
     <gazebo>
-    <plugin name="gazebo_ros_control" filename="libgazebo_ros_control.so">
-    </plugin>
+    	<plugin name="gazebo_ros_control" filename="libgazebo_ros_control.so">
+    	</plugin>
+  	</gazebo>
+  	<!-- camera -->
+  <gazebo reference="camera_link">
+  	<material>Gazebo/Green</material>
+    <sensor type="camera" name="camera1">
+      <update_rate>30.0</update_rate>
+      <camera name="head">
+        <horizontal_fov>1.3962634</horizontal_fov>
+        <image>
+          <width>800</width>
+          <height>800</height>
+          <format>R8G8B8</format>
+        </image>
+        <clip>
+          <near>0.02</near>
+          <far>300</far>
+        </clip>
+        <noise>
+          <type>gaussian</type>
+          <!-- Noise is sampled independently per pixel on each frame.
+               That pixel's noise value is added to each of its color
+               channels, which at that point lie in the range [0,1]. -->
+          <mean>0.0</mean>
+          <stddev>0.007</stddev>
+        </noise>
+      </camera>
+      <plugin name="camera_controller" filename="libgazebo_ros_camera.so">
+        <alwaysOn>true</alwaysOn>
+        <updateRate>0.0</updateRate>
+        <cameraName>rrbot/camera1</cameraName>
+        <imageTopicName>image_raw</imageTopicName>
+        <cameraInfoTopicName>camera_info</cameraInfoTopicName>
+        <frameName>camera_link</frameName>
+        <hackBaseline>0.07</hackBaseline>
+        <distortionK1>0.0</distortionK1>
+        <distortionK2>0.0</distortionK2>
+        <distortionK3>0.0</distortionK3>
+        <distortionT1>0.0</distortionT1>
+        <distortionT2>0.0</distortionT2>
+      </plugin>
+    </sensor>
   </gazebo>
 </robot>

File: urdf/robot_parameters.xacro (robot description, xacro)
@@ -7,3 +7,4 @@
   <xacro:property name="link_04_name" value="link_04" />
   <xacro:property name="link_05_name" value="link_05" />
+  <xacro:property name="camera_link" value="0.35" /> <!-- Size of square 'camera' box -->
 </robot>

Commit message: final robot model

File: urdf/links_joints.xacro (robot description, xacro)
@@ -32,5 +32,5 @@
     </transmission>
   </xacro:macro>
-  <xacro:macro name="m_link_cylinder" params="name origin_xyz origin_rpy radius length mass ixx ixy ixz iyy iyz izz">
+  <xacro:macro name="m_link_cylinder" params="name origin_xyz origin_rpy radius length mass ixx ixy ixz iyy iyz izz ">
     <link name="${name}">
       <inertial>
@@ -50,9 +50,9 @@
           <cylinder radius="${radius}" length="${length}" />
         </geometry>
-        <material name="cyan"/>
+        <material name="blue"/>
       </visual>
     </link>
   </xacro:macro>
-  <xacro:macro name="m_link_box" params="name origin_xyz origin_rpy size mass ixx ixy ixz iyy iyz izz">
+  <xacro:macro name="m_link_box" params="name origin_xyz origin_rpy size mass ixx ixy ixz iyy iyz izz ">
     <link name="${name}">
       <inertial>
@@ -72,5 +72,5 @@
           <box size="${size}" />
         </geometry>
-        <material name="blue"/>
+        <material name="cyan"/>
       </visual>
     </link>

File: urdf/mrm.xacro (robot description, xacro)
@@ -5,10 +5,55 @@
 <!-- this is fixed -->
 	<m_link_box name="${link_00_name}"
-              origin_rpy="0 0 0" origin_xyz="0 0 0"
+              origin_rpy="0 0 0" origin_xyz="0 0 0.4"
               mass="1024"
               ixx="170.667" ixy="0" ixz="0"
               iyy="170.667" iyz="0"
               izz="170.667"
-              size="1 1 1" />
+              size="1.5 1.5 0.3" />
+<!-- CHASSIS -->
+<!-- LEFT WHEEL -->
+<!-- <link name="left_wheel">
+        <pose>0.1 0.13 0.1 0 1.5707 1.5707</pose>
+        <collision name="collision">
+          <geometry>
+            <cylinder>
+              <radius>.1</radius>
+              <length>.05</length>
+            </cylinder>
+          </geometry>
+        </collision>
+        <visual name="visual">
+          <geometry>
+            <cylinder>
+              <radius>.1</radius>
+              <length>.05</length>
+            </cylinder>
+          </geometry>
+        </visual>
+      </link> -->
+<m_link_cylinder name="left_wheel"
+              origin_rpy="1.5708 0 0" origin_xyz="-0 -0.55 0"
+              mass="57.906"
+              ixx="12.679" ixy="0" ixz="0"
+              iyy="12.679" iyz="0"
+              izz="0.651"
+              radius="0.25" length="0.25" />
+<m_joint name="left_wheel__base_link" type="continuous"
+           axis_xyz="0 1 0"
+           origin_rpy="0 0 0" origin_xyz="0 0 -0.03"
+           parent="base_link" child="left_wheel"
+           limit_e="1000" limit_l="-3.14" limit_u="3.14" limit_v="0.5"/>
+<m_link_cylinder name="right_wheel"
+              origin_rpy="1.5708 0 0" origin_xyz="-0 0.55 0"
+              mass="57.906"
+              ixx="12.679" ixy="0" ixz="0"
+              iyy="12.679" iyz="0"
+              izz="0.651"
+              radius="0.25" length="0.25" />
+<m_joint name="right_wheel__base_link" type="continuous"
+           axis_xyz="0 1 0"
+           origin_rpy="0 0 0" origin_xyz="0 0 -0.03"
+           parent="base_link" child="right_wheel"
+           limit_e="1000" limit_l="-3.14" limit_u="3.14" limit_v="0.5"/>
 <!-- between the links there has to be a joint -->
 	<m_joint name="${link_00_name}__${link_01_name}" type="revolute"
@@ -76,5 +121,5 @@
     <joint name="camera_joint" type="fixed">
     	<axis xyz="0 1 0" />
-    	<origin rpy="0 0 0" xyz="0.7 0 0"/>
+    	<origin rpy="0 0 0" xyz="0.8 0 0.4"/>
     	<parent link="${link_00_name}"/>
     	<child link="camera_link"/>
@@ -83,5 +128,5 @@
   	<link name="camera_link">
     	<collision>
-      		<origin xyz="0.5 0 0" rpy="0 0 0"/>
+      		<origin xyz="0.8 0 0.4" rpy="0 0 0"/>
       		<geometry>
     			<box size="${camera_link} ${camera_link} ${camera_link}"/>

File: urdf/robot_parameters.xacro (robot description, xacro)
@@ -7,4 +7,4 @@
   <xacro:property name="link_04_name" value="link_04" />
   <xacro:property name="link_05_name" value="link_05" />
-  <xacro:property name="camera_link" value="0.35" /> <!-- Size of square 'camera' box -->
+  <xacro:property name="camera_link" value="0.2" /> <!-- Size of square 'camera' box -->
 </robot>

Commit message: final robot model wheels under the ground

File: urdf/links_joints.xacro (robot description, xacro)
@@ -29,4 +29,5 @@
         <hardwareInterface>hardware_interface/EffortJointInterface</hardwareInterface>
         <mechanicalReduction>1</mechanicalReduction>
+        <motorTorqueConstant>1.32</motorTorqueConstant>
       </actuator>
     </transmission>

File: urdf/original.xacro (robot description, xacro)
@@ -13,6 +13,25 @@
 <!-- CHASSIS -->
 <!-- LEFT WHEEL -->
+<!-- <link name="left_wheel">
+        <pose>0.1 0.13 0.1 0 1.5707 1.5707</pose>
+        <collision name="collision">
+          <geometry>
+            <cylinder>
+              <radius>.1</radius>
+              <length>.05</length>
+            </cylinder>
+          </geometry>
+        </collision>
+        <visual name="visual">
+          <geometry>
+            <cylinder>
+              <radius>.1</radius>
+              <length>.05</length>
+            </cylinder>
+          </geometry>
+        </visual>
+      </link> -->
 <m_link_cylinder name="left_wheel"
-              origin_rpy="1.5708 0 0" origin_xyz="-0 -0.55 0"
+              origin_rpy="1.5 0 0" origin_xyz="-0 -0.55 0"
               mass="57.906"
               ixx="12.679" ixy="0" ixz="0"
@@ -20,16 +39,4 @@
               izz="0.651"
               radius="0.25" length="0.25" />
-<gazebo reference="left_wheel">
-    <mu1 value="200.0" />
-    <mu2 value="100.0" />
-    <kp  value="5.0" />
-    <kd  value="1.0" />
-  </gazebo>
-  <gazebo reference="right_wheel">
-    <mu1 value="200.0" />
-    <mu2 value="100.0" />
-    <kp  value="5.0" />
-    <kd  value="1.0" />
-  </gazebo>
 <m_joint name="left_wheel__base_link" type="continuous"
            axis_xyz="0 1 0"
@@ -38,5 +45,5 @@
            limit_e="1000" limit_l="-3.14" limit_u="3.14" limit_v="0.5"/>
 <m_link_cylinder name="right_wheel"
-              origin_rpy="1.5708 0 0" origin_xyz="-0 0.55 0"
+              origin_rpy="1.5 0 0" origin_xyz="-0 0.55 0"
               mass="57.906"
               ixx="12.679" ixy="0" ixz="0"
@@ -63,5 +70,5 @@
               meshfile="package://mrm_decsription/meshes/Link1-v2.stl"
               meshscale="0.001 0.001 0.001" />
-	<m_joint name="${link_01_name}__${link_02_name}" type="revolute"
+	<m_joint name="${link_00_name}__${link_02_name}" type="revolute"
            axis_xyz="0 1 0"
            origin_rpy="0 0 0" origin_xyz="0 0 0.4"
@@ -110,155 +117,16 @@
               iyy="0.479" iyz="0"
               izz="0.204"
-              radius="0.15" length="0.25" />\
-     <!-- GRIPPER LINK AND LINK 5 JOINT -->
-    <joint name="joint4" type="revolute">
-		<parent link="${link_05_name}"/>
-		<child link="gripper_base"/>
-		<origin xyz="0 0 0.25" rpy="0 0 0"/>
-		<axis xyz="0 1 0"/>
-		<limit effort="100" velocity="100" lower="-1.5708" upper="1.5708"/>
-	</joint>
-	<transmission name="trans_joint4">
-      <type>transmission_interface/SimpleTransmission</type>
-      <joint name="joint4">
-        <hardwareInterface>hardware_interface/EffortJointInterface</hardwareInterface>
-      </joint>
-      <actuator name="motor_joint4">
-        <hardwareInterface>hardware_interface/EffortJointInterface</hardwareInterface>
-        <mechanicalReduction>1</mechanicalReduction>
-        <motorTorqueConstant>1.32</motorTorqueConstant>
-      </actuator>
-    </transmission>
-     <!-- GRIPPER LINK -->
-     <link name="gripper_base">
-	<collision>
-		<origin xyz="0 0 0" rpy="1.5708 0 0"/>
-		<geometry>
-			<cylinder length="0.4" radius="0.04"/>
-		</geometry>
-	</collision>
-	<visual>
-		<origin xyz="0 0 0" rpy="1.5708 0 0"/>
-		<geometry>
-			<cylinder length="0.4" radius="0.04"/>
-		</geometry>
-	</visual>
-	<inertial>
-		<origin xyz="0 0 0" rpy="1.5708 0 0"/>
-		<mass value="0.4"/>
-		<inertia
-			ixx="0.05" ixy="0.0" ixz="0.0"
-			iyy="0.002" iyz="0.0"
-			izz="0.05"/>
-	</inertial>
-</link>
-<gazebo reference="gripper_base">
-	<material>Gazebo/Red</material>
-</gazebo>
-<!-- The two main gripper rods -->
-<!-- IT HAS a prismatic joint -->
-<!-- translating along y axis -->
-<joint name="joint5" type="prismatic">
-	<parent link="gripper_base"/>
-	<child link="gripper_rod1"/>
-	<origin xyz="0 0.16 0" rpy="0 0 0"/>
-	<axis xyz="0 1 0"/>
-	<limit effort="100" velocity="100" lower="-0.16" upper="0.0"/>
-</joint>
-<transmission name="trans_joint5">
-      <type>transmission_interface/SimpleTransmission</type>
-      <joint name="joint5">
-        <hardwareInterface>hardware_interface/EffortJointInterface</hardwareInterface>
-      </joint>
-      <actuator name="motor_joint5">
-        <hardwareInterface>hardware_interface/EffortJointInterface</hardwareInterface>
-        <mechanicalReduction>1</mechanicalReduction>
-        <motorTorqueConstant>1.32</motorTorqueConstant>
-      </actuator>
-    </transmission>
-<!-- GRIPPER ROD 1 -->
-	<link name="gripper_rod1">
-	<collision>
-		<origin xyz="0 0 0.15" rpy="0 0 0"/>
-		<geometry>
-			<cylinder length="0.3" radius="0.04"/>
-		</geometry>
-	</collision>
-	<visual>
-		<origin xyz="0 0 0.15" rpy="0 0 0"/>
-		<geometry>
-			<cylinder length="0.3" radius="0.04"/>
-		</geometry>
-	</visual>
-	<inertial>
-		<origin xyz="0 0 0.15" rpy="0 0 0"/>
-		<mass value="0.2"/>
-		<inertia
-			ixx="0.02" ixy="0.0" ixz="0.0"
-			iyy="0.02" iyz="0.0"
-			izz="0.001"/>
-	</inertial>
-</link>
-<gazebo reference="gripper_rod1">
-	<material>Gazebo/Red</material>
-</gazebo>
-<!-- joint between gripper rod 2 and gripper base -->
-<!-- link6 and its prismatic joint6 relative to link4 -->
-<!-- translating along y axis -->
-<joint name="joint6" type="prismatic">
-	<parent link="gripper_base"/>
-	<child link="gripper_rod2"/>
-	<origin xyz="0 -0.16 0" rpy="0 0 0"/>
-	<axis xyz="0 1 0"/>
-	<limit effort="100" velocity="100" lower="0.0" upper="0.16"/>
-</joint>
-<transmission name="trans_joint6">
-      <type>transmission_interface/SimpleTransmission</type>
-      <joint name="joint6">
-        <hardwareInterface>hardware_interface/EffortJointInterface</hardwareInterface>
-      </joint>
-      <actuator name="motor_joint6">
-        <hardwareInterface>hardware_interface/EffortJointInterface</hardwareInterface>
-        <mechanicalReduction>1</mechanicalReduction>
-        <motorTorqueConstant>1.32</motorTorqueConstant>
-      </actuator>
-    </transmission>
+              radius="0.15" length="0.25" />
 <!-- camera link and joint -->
     <joint name="camera_joint" type="fixed">
     	<axis xyz="0 1 0" />
-    	<origin rpy="0 0 0" xyz="0.8 0 0.4"/>
+    	<origin rpy="0 0 0" xyz="0.7 0 0"/>
     	<parent link="${link_00_name}"/>
     	<child link="camera_link"/>
   	</joint>
- <!-- Link of gripper rod 2 -->
- 	<link name="gripper_rod2">
-	<collision>
-		<origin xyz="0 0 0.15" rpy="0 0 0"/>
-		<geometry>
-			<cylinder length="0.3" radius="0.04"/>
-		</geometry>
-	</collision>
-	<visual>
-		<origin xyz="0 0 0.15" rpy="0 0 0"/>
-		<geometry>
-			<cylinder length="0.3" radius="0.04"/>
-		</geometry>
-	</visual>
-	<inertial>
-		<origin xyz="0 0 0.15" rpy="0 0 0"/>
-		<mass value="0.2"/>
-		<inertia
-			ixx="0.02" ixy="0.0" ixz="0.0"
-			iyy="0.02" iyz="0.0"
-			izz="0.001"/>
-	</inertial>
-</link>
-<gazebo reference="gripper_rod2">
-	<material>Gazebo/Red</material>
-</gazebo>
  	 <!-- Camera -->
   	<link name="camera_link">
     	<collision>
-      		<origin xyz="0.8 0 0.4" rpy="0 0 0"/>
+      		<origin xyz="0.5 0 0" rpy="0 0 0"/>
       		<geometry>
     			<box size="${camera_link} ${camera_link} ${camera_link}"/>
